Commit message: now work p2

File: franka_description/robots/hand.xacro (robot description, xacro)
@@ -12,5 +12,5 @@
       <visual>
         <geometry>
-          <mesh filename="package://franka_description/meshes/visual/FTSensorPlusWiderLineEndEffector.dae"/> <!-- changed by ORION and NEEL -->
+          <mesh filename="package://pbal/franka_description/meshes/visual/FTSensorPlusWiderLineEndEffector.dae"/> <!-- changed by ORION and NEEL -->
         </geometry>
         <origin rpy="3.1416 0 0.7853" xyz="-0.012 0 -0.0945" />
@@ -18,5 +18,5 @@
       <collision>
         <geometry>
-          <mesh filename="package://franka_description/meshes/collision/hand.stl"/>
+          <mesh filename="package://pbal/franka_description/meshes/visual/FTSensorPlusWiderLineEndEffector.dae"/>
         </geometry>
       </collision>

File: franka_description/robots/panda_arm.urdf.xacro (robot description, xacro)
@@ -1,5 +1,5 @@
 <?xml version='1.0' encoding='utf-8'?>
 <robot xmlns:xacro="http://www.ros.org/wiki/xacro" name="panda">
-  <xacro:include filename="$(find franka_description)/robots/panda_arm.xacro" />
+  <xacro:include filename="$(find pbal)/franka_description/robots/panda_arm.xacro" />
   <xacro:panda_arm />
 </robot>

File: franka_description/robots/panda_arm.xacro (robot description, xacro)
@@ -1,5 +1,5 @@
 <?xml version='1.0' encoding='utf-8'?>
 <robot xmlns:xacro="http://www.ros.org/wiki/xacro" name="panda">
-  <xacro:macro name="panda_arm" params="arm_id:='panda' description_pkg:='franka_description' connected_to:='' xyz:='0 0 0' rpy:='0 0 0'">
+  <xacro:macro name="panda_arm" params="arm_id:='panda' description_pkg:='pbal' connected_to:='' xyz:='0 0 0' rpy:='0 0 0'">
     <xacro:unless value="${not connected_to}">
       <joint name="${arm_id}_joint_${connected_to}" type="fixed">
@@ -12,10 +12,10 @@
       <visual>
         <geometry>
-          <mesh filename="package://${description_pkg}/meshes/visual/link0.dae"/>
+          <mesh filename="package://${description_pkg}/franka_description/meshes/visual/link0.dae"/>
         </geometry>
       </visual>
       <collision>
         <geometry>
-          <mesh filename="package://${description_pkg}/meshes/collision/link0.stl"/>
+          <mesh filename="package://${description_pkg}/franka_description/meshes/collision/link0.stl"/>
         </geometry>
       </collision>
@@ -24,10 +24,10 @@
       <visual>
         <geometry>
-          <mesh filename="package://${description_pkg}/meshes/visual/link1.dae"/>
+          <mesh filename="package://${description_pkg}/franka_description/meshes/visual/link1.dae"/>
         </geometry>
       </visual>
       <collision>
         <geometry>
-          <mesh filename="package://${description_pkg}/meshes/collision/link1.stl"/>
+          <mesh filename="package://${description_pkg}/franka_description/meshes/collision/link1.stl"/>
         </geometry>
       </collision>
@@ -44,10 +44,10 @@
       <visual>
         <geometry>
-          <mesh filename="package://${description_pkg}/meshes/visual/link2.dae"/>
+          <mesh filename="package://${description_pkg}/franka_description/meshes/visual/link2.dae"/>
         </geometry>
       </visual>
       <collision>
         <geometry>
-          <mesh filename="package://${description_pkg}/meshes/collision/link2.stl"/>
+          <mesh filename="package://${description_pkg}/franka_description/meshes/collision/link2.stl"/>
         </geometry>
       </collision>
@@ -64,10 +64,10 @@
       <visual>
         <geometry>
-          <mesh filename="package://${description_pkg}/meshes/visual/link3.dae"/>
+          <mesh filename="package://${description_pkg}/franka_description/meshes/visual/link3.dae"/>
         </geometry>
       </visual>
       <collision>
         <geometry>
-          <mesh filename="package://${description_pkg}/meshes/collision/link3.stl"/>
+          <mesh filename="package://${description_pkg}/franka_description/meshes/collision/link3.stl"/>
         </geometry>
       </collision>
@@ -84,10 +84,10 @@
       <visual>
         <geometry>
-          <mesh filename="package://${description_pkg}/meshes/visual/link4.dae"/>
+          <mesh filename="package://${description_pkg}/franka_description/meshes/visual/link4.dae"/>
         </geometry>
       </visual>
       <collision>
         <geometry>
-          <mesh filename="package://${description_pkg}/meshes/collision/link4.stl"/>
+          <mesh filename="package://${description_pkg}/franka_description/meshes/collision/link4.stl"/>
         </geometry>
       </collision>
@@ -104,10 +104,10 @@
       <visual>
         <geometry>
-          <mesh filename="package://${description_pkg}/meshes/visual/link5.dae"/>
+          <mesh filename="package://${description_pkg}/franka_description/meshes/visual/link5.dae"/>
         </geometry>
       </visual>
       <collision>
         <geometry>
-          <mesh filename="package://${description_pkg}/meshes/collision/link5.stl"/>
+          <mesh filename="package://${description_pkg}/franka_description/meshes/collision/link5.stl"/>
         </geometry>
       </collision>
@@ -124,10 +124,10 @@
       <visual>
         <geometry>
-          <mesh filename="package://${description_pkg}/meshes/visual/link6.dae"/>
+          <mesh filename="package://${description_pkg}/franka_description/meshes/visual/link6.dae"/>
         </geometry>
       </visual>
       <collision>
         <geometry>
-          <mesh filename="package://${description_pkg}/meshes/collision/link6.stl"/>
+          <mesh filename="package://${description_pkg}/franka_description/meshes/collision/link6.stl"/>
         </geometry>
       </collision>
@@ -144,10 +144,10 @@
       <visual>
         <geometry>
-          <mesh filename="package://${description_pkg}/meshes/visual/link7.dae"/>
+          <mesh filename="package://${description_pkg}/franka_description/meshes/visual/link7.dae"/>
         </geometry>
       </visual>
       <collision>
         <geometry>
-          <mesh filename="package://${description_pkg}/meshes/collision/link7.stl"/>
+          <mesh filename="package://${description_pkg}/franka_description/meshes/collision/link7.stl"/>
         </geometry>
       </collision>

File: franka_description/robots/panda_arm_hand.urdf.xacro (robot description, xacro)
@@ -1,6 +1,6 @@
 <?xml version="1.0" encoding="utf-8"?>
 <robot xmlns:xacro="http://www.ros.org/wiki/xacro" name="panda">
-  <xacro:include filename="$(find franka_description)/robots/panda_arm.xacro"/>
-  <xacro:include filename="$(find franka_description)/robots/hand.xacro"/>
+  <xacro:include filename="$(find pbal)/franka_description/robots/panda_arm.xacro"/>
+  <xacro:include filename="$(find pbal)/franka_description/robots/hand.xacro"/>
   <xacro:panda_arm />
   <xacro:hand ns="panda" rpy="0 0 ${-pi/4}" connected_to="panda_link8"/>
